Commit message: feat: change to use ESP32 from PICO

File: edge/workspace/src/amr_description/urdf/turtlebot3_burger.urdf (robot description, URDF)
Before this commit: robot turtlebot3_burger, 7 links, 6 joints
Joints:
- joint ${namespace}wheel_left_joint: origin xyz=0.0 0.08 0.023 rpy=-1.57 0 0 -> xyz=0.0 0.1475 0.023 rpy=-1.57 0 0
- joint ${namespace}wheel_right_joint: origin xyz=0.0 -0.080 0.023 rpy=-1.57 0 0 -> xyz=0.0 -0.1475 0.023 rpy=-1.57 0 0
