Commit message: feat: add SO-101 arm and HP60C RGB-D camera to robot model and simulation

File: edge/workspace/src/amr_description/urdf/amr.urdf.xacro (robot description, xacro)
@@ -1,8 +1,31 @@
 <?xml version="1.0"?>
 <robot name="amr" xmlns:xacro="http://www.ros.org/wiki/xacro">
+    <xacro:arg name="namespace" default=""/>
+    <xacro:property name="namespace" value="$(arg namespace)"/>
     <xacro:include filename="common_properties.xacro" />
-    <xacro:include filename="turtlebot3_burger.urdf" />
-    <xacro:include filename="imx708_camera.urdf" />
-    <xacro:include filename="imx708_camera_gazebo.urdf" />
+    <xacro:include filename="chassis_base.urdf.xacro" />
+    <xacro:include filename="so101_new_calib.urdf.xacro" />
+    <xacro:include filename="nuwa_hp60c.urdf.xacro" />
+    <xacro:include filename="nuwa_hp60c_gazebo.urdf.xacro" />
     <xacro:include filename="ros2_control.urdf" />
+    <joint name="${namespace}arm_mount_joint" type="fixed">
+        <origin xyz="-0.047 0 0.0915" rpy="0 0 0"/>
+        <parent link="${namespace}base_link"/>
+        <child link="${namespace}arm_mount_link"/>
+    </joint>
+    <link name="${namespace}arm_mount_link">
+        <visual>
+            <origin xyz="0 0 0" rpy="0 0 0"/>
+            <geometry>
+                <mesh filename="package://amr_description/meshes/arm_mount.stl" scale="0.0001 0.0001 0.0001"/>
+            </geometry>
+            <material name="dark"/>
+        </visual>
+    </link>
+    <!-- SO101のarm_base_linkは原点が台座底面より2.4mm上にあるため、台座の厚み(9.9mm)に足す。 -->
+    <joint name="${namespace}arm_base_joint" type="fixed">
+        <origin xyz="-0.021 0 0.01" rpy="0 0 0"/>
+        <parent link="${namespace}arm_mount_link"/>
+        <child link="${namespace}arm_base_link"/>
+    </joint>
 </robot>

File: edge/workspace/src/amr_description/urdf/common_properties.xacro (robot description, xacro)
@@ -32,3 +32,10 @@
     <color rgba="1.0 1.0 1.0 1.0"/>
   </material>
+  <!-- For SO101 -->
+  <material name="3d_printed">
+    <color rgba="1.0 0.82 0.12 1.0"/>
+  </material>
+  <material name="sts3215">
+    <color rgba="0.1 0.1 0.1 1.0"/>
+  </material>
 </robot>

Commit message: feat: drive the real SO-101 arm from MoveIt with auto-start, standby pose and collision geometry

File: edge/workspace/src/amr_description/urdf/amr.urdf.xacro (robot description, xacro)
@@ -11,4 +11,9 @@
         <xacro:include filename="nuwa_hp60c_gazebo.urdf.xacro" />
         <xacro:include filename="ros2_control.urdf" />
+    </xacro:if>
+    <!-- 実機のSO-101をros2_controlで動かす時だけtrueにする(use_gazeboはfalseにすること)。 -->
+    <xacro:arg name="use_real_arm" default="false"/>
+    <xacro:if value="$(arg use_real_arm)">
+        <xacro:include filename="so101_feetech.ros2_control.xacro" />
     </xacro:if>
     <joint name="${namespace}arm_mount_joint" type="fixed">
@@ -25,4 +30,10 @@
             <material name="dark"/>
         </visual>
+        <collision>
+            <origin xyz="0 0 0" rpy="0 0 0"/>
+            <geometry>
+                <mesh filename="package://amr_description/meshes/arm_mount.stl" scale="0.0001 0.0001 0.0001"/>
+            </geometry>
+        </collision>
     </link>
     <!-- SO101のarm_base_linkは原点が台座底面より2.4mm上にあるため、台座の厚み(9.9mm)に足す。 -->

File: edge/workspace/src/amr_description/urdf/nuwa_hp60c.urdf.xacro (robot description, xacro)
@@ -22,4 +22,10 @@
       <material name="3d_printed"/>
     </visual>
+    <collision>
+      <origin xyz="0 0 0" rpy="0 0 0"/>
+      <geometry>
+        <mesh filename="package://amr_description/meshes/arm_camera_mount.stl" scale="0.001 0.001 0.001"/>
+      </geometry>
+    </collision>
   </link>
   <joint name="hp60c_joint" type="fixed">
@@ -36,4 +42,10 @@
       <material name="dark"/>
     </visual>
+    <collision>
+      <origin xyz="-0.0105 -0.0023 0" rpy="0 0 0"/>
+      <geometry>
+        <box size="0.029 0.090 0.019"/>
+      </geometry>
+    </collision>
   </link>
   <!-- ドライバ(ascamera)は画像・点群をこのフレームの子(camera_color_0等)としてTFを出すため、名前を合わせる。
